Commit message: Parameterize some parameters.

File: description/gunnar.urdf.xacro (robot description, xacro)
@@ -1,4 +1,5 @@
 <?xml version="1.0" encoding="UTF-8"?>
 <robot name="gunnar" xmlns:xacro="http://ros.org/wiki/xacro">
+     <!-- ================= MACROS ============== -->
        <xacro:macro name="inertialEye" params="ma mo">
             <inertial>
@@ -38,14 +39,30 @@
             </visual>
         </xacro:macro>
+    <!-- ============== DIMENSIONS ================ -->
+    <xacro:property name="CHASSISLENGTH" value=".28" />
+    <xacro:property name="CHASSISHEIGHT" value=".165" />
+    <xacro:property name="CHASSISWIDTH" value=".19" />
+    <xacro:property name="BRACKETLENGTH" value=".1" />
+    <xacro:property name="CLEARANCE" value=".06" />
+    <xacro:property name="CASTERBRACKETHEIGHT" value="-${CHASSISHEIGHT/2-.055}" />
+    <xacro:property name="CASTERARMLENGTH" value=".085" />
+    <xacro:property name="SHEETMETALTHICKNESS" value=".003" />
+    <xacro:property name="SIDEWHEELMASS" value=".165" />
+    <xacro:property name="CASTERMASS" value=".695" />
+    <xacro:property name="LIDARMASS" value=".1" />
+    <xacro:property name="CHASSISMASS" value="${4.922 - 2*SIDEWHEELMASS - CASTERMASS - LIDARMASS}" />
+    <xacro:property name="wheelFriction" value="0.5" />
+    <xacro:property name="wheelDamping" value="0.5" />
+    <xacro:property name="M_PI" value="3.1415926535897931" />
     <!-- ============= BODY ======= -->
     <link name="chassis">
-        <origin xyz="0 0 .17416"/>
-        <xacro:inertialEye ma="1" mo=".005" />
-        <xacro:macbox size=".3048 .1742 .1742" name="chassis">
+        <origin xyz="0 0 ${CLEARANCE}"/>
+        <xacro:inertialEye ma="${CHASSISMASS}" mo=".005" />
+        <xacro:macbox size="${CHASSISLENGTH} ${CHASSISWIDTH} ${CHASSISHEIGHT}" name="chassis">
             <origin xyz="0 0 0"/>
             <material name="plastic"/>
         </xacro:macbox>
-        <xacro:macbox size=".08708 .04354 .0254" name="caster_bracket">
-            <origin xyz="-.1959 0 0" />
+        <xacro:macbox size="${BRACKETLENGTH} .035 ${SHEETMETALTHICKNESS}" name="caster_bracket">
+            <origin xyz="-${(BRACKETLENGTH+CHASSISLENGTH)/2} 0 ${CASTERBRACKETHEIGHT}" />
             <material name="steel">
               <ambient>.5 .5 .5 1"</ambient>
@@ -65,6 +82,6 @@
           <surface />
         </xacro:maccyl>
-        <xacro:macbox size=".14 .01 .04" name="caster_arm_l">
-            <origin xyz="-0.04053 -.03 -.06" rpy="0 -1 0" />
+        <xacro:macbox size="${CASTERARMLENGTH} ${SHEETMETALTHICKNESS} .04" name="caster_arm_l">
+            <origin xyz="-0.04053 -.02 -.04" rpy="0 -1 0" />
             <material name="steel">
               <ambient>.5 .5 .5 1</ambient>
@@ -74,6 +91,6 @@
             </material>
         </xacro:macbox>
-        <xacro:macbox size=".14 .01 .04" name="caster_arm_l">
-            <origin xyz="-0.04053 .03 -.06" rpy="0 -1 0" />
+        <xacro:macbox size="${CASTERARMLENGTH} ${SHEETMETALTHICKNESS} .04" name="caster_arm_l">
+            <origin xyz="-0.04053 .02 -.04" rpy="0 -1 0" />
             <material name="steel">
               <ambient>.5 .5 .5 1</ambient>
@@ -87,6 +104,6 @@
         <link name="left_wheel">
             <origin />
-            <xacro:inertialEye ma=".1" mo=".005" />
-            <xacro:maccyl radius=".06531" length=".05" name="left_wheel">
+            <xacro:inertialEye ma="${SIDEWHEELMASS}" mo="${SIDEWHEELMASS*.04*.04}" />
+            <xacro:maccyl radius=".05" length=".025" name="left_wheel">
                 <origin />
                   <material name="rubber">
@@ -107,6 +124,6 @@
         <link name="right_wheel">
             <origin />
-            <xacro:inertialEye ma=".1" mo=".005" />
-            <xacro:maccyl radius=".06531" length=".05" name="right_wheel">
+            <xacro:inertialEye ma="${SIDEWHEELMASS}" mo="${SIDEWHEELMASS*.04*.04}" />
+            <xacro:maccyl radius=".05" length=".025" name="right_wheel">
                 <origin />
                   <material name="rubber">
@@ -127,6 +144,6 @@
         <link name="caster_wheel">
             <origin />
-            <xacro:inertialEye ma=".1" mo=".005" />
-            <xacro:maccyl radius=".06531" length=".05" name="caster_wheel">
+            <xacro:inertialEye ma="${CASTERMASS}" mo="${.695*.04*.04}" />
+            <xacro:maccyl radius=".05" length=".025" name="caster_wheel">
                 <origin />
                   <material name="rubber">
@@ -147,6 +164,6 @@
         <link name="lidar_disk">
             <origin />
-            <xacro:inertialEye ma=".1" mo=".005" />
-            <xacro:maccyl radius=".06531" length=".05" name="lidar_disk">
+            <xacro:inertialEye ma="${LIDARMASS}" mo="${LIDARMASS*.04*.04}" />
+            <xacro:maccyl radius=".04" length=".025" name="lidar_disk">
                 <origin />
                   <material name="rubber">
@@ -166,5 +183,4 @@
         </link>
         <!-- ============= JOINTS ============== -->
-        <xacro:property name="M_PI" value="3.1415926535897931" />
         <xacro:macro name="continuousJoint" params="name posexyz poserpy parent child xyz friction damping">
             <joint type="continuous" name="${name}_continuous_joint">
@@ -186,6 +202,4 @@
             </joint>
         </xacro:macro>
-        <xacro:property name="wheelFriction" value="0.5" />
-        <xacro:property name="wheelDamping" value="0.5" />
         <xacro:continuousJoint name="left_wheel"
             posexyz="0 -.12 -.11" poserpy="-${M_PI / 2} 0 0"
@@ -197,5 +211,5 @@
             friction="${wheelFriction}" damping="${wheelDamping}" />
         <xacro:continuousJoint name="caster_wheel"
-            posexyz="-.05 0 -.11" poserpy="${M_PI / 2} 0 0"
+            posexyz="-.04 0 -.085" poserpy="${M_PI / 2} 0 0"
             parent="caster_arm" child="caster_wheel" xyz="0 0 1"
             friction="${wheelFriction}" damping="${wheelDamping}" />
@@ -205,9 +219,10 @@
             friction=".001" damping=".001" />
         <xacro:revoluteJoint name="caster_yaw"
-            posexyz="-.23947 0 0"  poserpy="0 0 0"
+            posexyz="-.23947 0 ${CASTERBRACKETHEIGHT}"  poserpy="0 0 0"
             parent="chassis" child="caster_arm" xyz="0 0 1"
             friction=".1" damping=".1"
-            lower="-${M_PI/8}" upper="${M_PI/8}"
+            lower="-${M_PI}" upper="${M_PI}"
             effort="1000" velocity="1000" />
+    <!-- =================== PLUGINS ================= -->
     <gazebo>
         <plugin name="p3d" filename="libgazebo_ros_p3d.so">

Commit message: Make movement a little more realistic.

File: description/gunnar.urdf.xacro (robot description, xacro)
@@ -48,10 +48,18 @@
     <xacro:property name="CASTERARMLENGTH" value=".085" />
     <xacro:property name="SHEETMETALTHICKNESS" value=".003" />
+    <xacro:property name="WHEELRADIUS" value=".05" />
+    <xacro:property name="WHEELLENGTH" value=".025" />
     <xacro:property name="SIDEWHEELMASS" value=".165" />
     <xacro:property name="CASTERMASS" value=".695" />
     <xacro:property name="LIDARMASS" value=".1" />
     <xacro:property name="CHASSISMASS" value="${4.922 - 2*SIDEWHEELMASS - CASTERMASS - LIDARMASS}" />
-    <xacro:property name="wheelFriction" value="0.5" />
-    <xacro:property name="wheelDamping" value="0.5" />
+    <xacro:property name="WHEELJOINTFRICTION" value="0.5" />
+    <xacro:property name="WHEELJOINTDAMPING" value="0.5" />
+    <xacro:property name="WHEELSURFACEFRICTION" value=".9" />
+    <xacro:property name="WHEELSURFACESLIP" value="0.1" />
+    <xacro:property name="WHEELTORQUE" value=".2" />
+    <xacro:property name="WHEELACCEL" value=".2" />
+    <xacro:property name="CASTERJOINTDAMPING" value=".1" />
+    <xacro:property name="CASTERJOINTFRICTION" value=".1" />
     <xacro:property name="M_PI" value="3.1415926535897931" />
     <!-- ============= BODY ======= -->
@@ -82,6 +90,9 @@
           <surface />
         </xacro:maccyl>
+        <xacro:property name="CASTERARMX" value="-.04053" />
+        <xacro:property name="CASTERARMYabs" value=".02" />
+        <xacro:property name="CASTERARMZ" value="-.04" />
         <xacro:macbox size="${CASTERARMLENGTH} ${SHEETMETALTHICKNESS} .04" name="caster_arm_l">
-            <origin xyz="-0.04053 -.02 -.04" rpy="0 -1 0" />
+            <origin xyz="${CASTERARMX} -${CASTERARMYabs} ${CASTERARMZ}" rpy="0 -1 0" />
             <material name="steel">
               <ambient>.5 .5 .5 1</ambient>
@@ -92,5 +103,5 @@
         </xacro:macbox>
         <xacro:macbox size="${CASTERARMLENGTH} ${SHEETMETALTHICKNESS} .04" name="caster_arm_l">
-            <origin xyz="-0.04053 .02 -.04" rpy="0 -1 0" />
+            <origin xyz="${CASTERARMX} ${CASTERARMYabs} ${CASTERARMZ}" rpy="0 -1 0" />
             <material name="steel">
               <ambient>.5 .5 .5 1</ambient>
@@ -105,16 +116,16 @@
             <origin />
             <xacro:inertialEye ma="${SIDEWHEELMASS}" mo="${SIDEWHEELMASS*.04*.04}" />
-            <xacro:maccyl radius=".05" length=".025" name="left_wheel">
-                <origin />
-                  <material name="rubber">
-                    <ambient>0 0 0 1</ambient>
-                  </material>
-                <surface>
-                    <friction>
-                        <ode>
-                            <mu>.9</mu>
-                            <mu2>.9</mu2>
-                            <slip1>.1</slip1>
-                            <slip2>.1</slip2>
+            <xacro:maccyl radius="${WHEELRADIUS}" length="${WHEELLENGTH}" name="left_wheel">
+                <origin />
+                  <material name="rubber">
+                    <ambient>0 0 0 1</ambient>
+                  </material>
+                <surface>
+                    <friction>
+                        <ode>
+                            <mu>${WHEELSURFACEFRICTION}</mu>
+                            <mu2>${WHEELSURFACEFRICTION}</mu2>
+                            <slip1>${WHEELSURFACESLIP}</slip1>
+                            <slip2>${WHEELSURFACESLIP}</slip2>
                         </ode>
                     </friction>
@@ -125,16 +136,16 @@
             <origin />
             <xacro:inertialEye ma="${SIDEWHEELMASS}" mo="${SIDEWHEELMASS*.04*.04}" />
-            <xacro:maccyl radius=".05" length=".025" name="right_wheel">
-                <origin />
-                  <material name="rubber">
-                    <ambient>0 0 0 1</ambient>
-                  </material>
-                <surface>
-                    <friction>
-                        <ode>
-                            <mu>.9</mu>
-                            <mu2>.9</mu2>
-                            <slip1>.1</slip1>
-                            <slip2>.1</slip2>
+            <xacro:maccyl radius="${WHEELRADIUS}" length="${WHEELLENGTH}" name="right_wheel">
+                <origin />
+                  <material name="rubber">
+                    <ambient>0 0 0 1</ambient>
+                  </material>
+                <surface>
+                    <friction>
+                        <ode>
+                            <mu>${WHEELSURFACEFRICTION}</mu>
+                            <mu2>${WHEELSURFACEFRICTION}</mu2>
+                            <slip1>${WHEELSURFACESLIP}</slip1>
+                            <slip2>${WHEELSURFACESLIP}</slip2>
                         </ode>
                     </friction>
@@ -145,16 +156,16 @@
             <origin />
             <xacro:inertialEye ma="${CASTERMASS}" mo="${.695*.04*.04}" />
-            <xacro:maccyl radius=".05" length=".025" name="caster_wheel">
-                <origin />
-                  <material name="rubber">
-                    <ambient>0 0 0 1</ambient>
-                  </material>
-                <surface>
-                    <friction>
-                        <ode>
-                            <mu>.9</mu>
-                            <mu2>.9</mu2>
-                            <slip1>.1</slip1>
-                            <slip2>.1</slip2>
+            <xacro:maccyl radius="${WHEELRADIUS}" length="${WHEELLENGTH}" name="caster_wheel">
+                <origin />
+                  <material name="rubber">
+                    <ambient>0 0 0 1</ambient>
+                  </material>
+                <surface>
+                    <friction>
+                        <ode>
+                            <mu>${WHEELSURFACEFRICTION}</mu>
+                            <mu2>${WHEELSURFACEFRICTION}</mu2>
+                            <slip1>${WHEELSURFACESLIP}</slip1>
+                            <slip2>${WHEELSURFACESLIP}</slip2>
                         </ode>
                     </friction>
@@ -205,13 +216,13 @@
             posexyz="0 -.12 -.11" poserpy="-${M_PI / 2} 0 0"
             parent="chassis" child="left_wheel" xyz="0 0 1"
-            friction="${wheelFriction}" damping="${wheelDamping}" />
+            friction="${WHEELJOINTFRICTION}" damping="${WHEELJOINTDAMPING}" />
         <xacro:continuousJoint name="right_wheel"
             posexyz="0 .12 -.11" poserpy="-${M_PI / 2} 0 0"
             parent="chassis" child="right_wheel" xyz="0 0 1"
-            friction="${wheelFriction}" damping="${wheelDamping}" />
+            friction="${WHEELJOINTFRICTION}" damping="${WHEELJOINTDAMPING}" />
         <xacro:continuousJoint name="caster_wheel"
             posexyz="-.04 0 -.085" poserpy="${M_PI / 2} 0 0"
             parent="caster_arm" child="caster_wheel" xyz="0 0 1"
-            friction="${wheelFriction}" damping="${wheelDamping}" />
+            friction="${WHEELJOINTFRICTION}" damping="${WHEELJOINTDAMPING}" />
         <xacro:continuousJoint name="lidar_disk"
             posexyz="0 0 .12" poserpy="0 0 0"
@@ -221,5 +232,5 @@
             posexyz="-.23947 0 ${CASTERBRACKETHEIGHT}"  poserpy="0 0 0"
             parent="chassis" child="caster_arm" xyz="0 0 1"
-            friction=".1" damping=".1"
+            friction="${CASTERJOINTFRICTION}" damping="${CASTERJOINTDAMPING}"
             lower="-${M_PI}" upper="${M_PI}"
             effort="1000" velocity="1000" />
@@ -245,8 +256,10 @@
             <leftJoint>left_wheel_continuous_joint</leftJoint>
             <rightJoint>right_wheel_continuous_joint</rightJoint>
-            <wheelSeparation>0.2242</wheelSeparation>
-            <wheelDiameter>.06531</wheelDiameter>
-            <wheelTorque>.02</wheelTorque>
-            <wheelAcceleration>.1</wheelAcceleration>
+            <!-- <wheelSeparation>0.2242</wheelSeparation> -->
+            <!-- <wheelDiameter>.06531</wheelDiameter> -->
+            <wheelSeparation>${CHASSISWIDTH+WHEELLENGTH}</wheelSeparation>
+            <wheelDiameter>${2*WHEELRADIUS}</wheelDiameter>
+            <wheelTorque>${WHEELTORQUE}</wheelTorque>
+            <wheelAcceleration>${WHEELACCEL}</wheelAcceleration>
             <odometryTopic>odom</odometryTopic>
             <odometryFrame>odom</odometryFrame>
