Commit message: Reformat description XML.

File: description/gunnar.urdf.xacro (robot description, xacro)
@@ -1,43 +1,44 @@
 <?xml version="1.0" encoding="UTF-8"?>
-<robot name="gunnar" xmlns:xacro="http://ros.org/wiki/xacro">
-     <!-- ================= MACROS ============== -->
-       <xacro:macro name="inertialEye" params="ma mo">
-            <inertial>
-                <mass value="${ma}" />
-                <inertia ixx="${mo}" iyy="${mo}" izz="${mo}" ixy="0" ixz="0" iyz="0" />
-            </inertial>
-        </xacro:macro>
-        <xacro:macro name="macbox" params="size name *origin *material">
-            <collision name="${name}_collision">
-                <xacro:insert_block name="origin" />
-                <geometry>
-                    <box size="${size}" />
-                </geometry>
-            </collision>
-            <visual name="${name}_visual">
-                <xacro:insert_block name="origin" />
-                <geometry>
-                    <box size="${size}" />
-                </geometry>
-                <xacro:insert_block name="material" />
-            </visual>
-        </xacro:macro>
-        <xacro:macro name="maccyl" params="radius length name *origin *material *surface">
-            <collision name="${name}_collision">
-              <xacro:insert_block name="origin" />
-                <geometry>
-                    <cylinder radius="${radius}" length="${length}" />
-                </geometry>
-                <xacro:insert_block name="surface"/>
-            </collision>
-            <visual name="${name}_visual">
-              <xacro:insert_block name="origin" />
-                <geometry>
-                    <cylinder radius="${radius}" length="${length}" />
-                </geometry>
-                <xacro:insert_block name="material"/>
-            </visual>
-        </xacro:macro>
-    <!-- ============== DIMENSIONS ================ -->
+<robot name="gunnar"
+    xmlns:xacro="http://ros.org/wiki/xacro">
+    <!-- ============== MACROS ============== -->
+    <xacro:macro name="inertialEye" params="ma mo">
+        <inertial>
+            <mass value="${ma}" />
+            <inertia ixx="${mo}" iyy="${mo}" izz="${mo}" ixy="0" ixz="0" iyz="0" />
+        </inertial>
+    </xacro:macro>
+    <xacro:macro name="macbox" params="size name *origin *material">
+        <collision name="${name}_collision">
+            <xacro:insert_block name="origin" />
+            <geometry>
+                <box size="${size}" />
+            </geometry>
+        </collision>
+        <visual name="${name}_visual">
+            <xacro:insert_block name="origin" />
+            <geometry>
+                <box size="${size}" />
+            </geometry>
+            <xacro:insert_block name="material" />
+        </visual>
+    </xacro:macro>
+    <xacro:macro name="maccyl" params="radius length name *origin *material *surface">
+        <collision name="${name}_collision">
+            <xacro:insert_block name="origin" />
+            <geometry>
+                <cylinder radius="${radius}" length="${length}" />
+            </geometry>
+            <xacro:insert_block name="surface"/>
+        </collision>
+        <visual name="${name}_visual">
+            <xacro:insert_block name="origin" />
+            <geometry>
+                <cylinder radius="${radius}" length="${length}" />
+            </geometry>
+            <xacro:insert_block name="material"/>
+        </visual>
+    </xacro:macro>
+    <!-- ============== DIMENSIONS ============== -->
     <xacro:property name="CHASSISLENGTH" value=".28" />
     <xacro:property name="CHASSISHEIGHT" value=".165" />
@@ -74,19 +75,19 @@
             <origin xyz="-${(BRACKETLENGTH+CHASSISLENGTH)/2} 0 ${CASTERBRACKETHEIGHT}" />
             <material name="steel">
-              <ambient>.5 .5 .5 1"</ambient>
-              <diffuse>0 0 0 1</diffuse>
-              <specular>0.1 0.1 0.1 1</specular>
-              <emissive>0 0 0 0</emissive>
-            </material>
-        </xacro:macbox>
-    </link>
-      <!-- ============= CASTER ARM =============== -->
-      <link name="caster_arm">
+                <ambient>.5 .5 .5 1"</ambient>
+                <diffuse>0 0 0 1</diffuse>
+                <specular>0.1 0.1 0.1 1</specular>
+                <emissive>0 0 0 0</emissive>
+            </material>
+        </xacro:macbox>
+    </link>
+    <!-- ============== CASTER ARM ============== -->
+    <link name="caster_arm">
         <origin />
         <xacro:inertialEye ma=".1" mo=".005" />
         <xacro:maccyl radius=".02" length=".02" name="caster_yawjoint">
-          <origin xyz="0 0 0" />
-          <material  name="steel"/>
-          <surface />
+            <origin xyz="0 0 0" />
+            <material  name="steel"/>
+            <surface />
         </xacro:maccyl>
         <xacro:property name="CASTERARMX" value="-.04053" />
@@ -96,8 +97,8 @@
             <origin xyz="${CASTERARMX} -${CASTERARMYabs} ${CASTERARMZ}" rpy="0 -1 0" />
             <material name="steel">
-              <ambient>.5 .5 .5 1</ambient>
-              <diffuse>0 0 0 1</diffuse>
-              <specular>0.1 0.1 0.1 1</specular>
-              <emissive>0 0 0 0</emissive>
+                <ambient>.5 .5 .5 1</ambient>
+                <diffuse>0 0 0 1</diffuse>
+                <specular>0.1 0.1 0.1 1</specular>
+                <emissive>0 0 0 0</emissive>
             </material>
         </xacro:macbox>
@@ -105,129 +106,129 @@
             <origin xyz="${CASTERARMX} ${CASTERARMYabs} ${CASTERARMZ}" rpy="0 -1 0" />
             <material name="steel">
-              <ambient>.5 .5 .5 1</ambient>
-              <diffuse>0 0 0 1</diffuse>
-              <specular>0.1 0.1 0.1 1</specular>
-              <emissive>0 0 0 0</emissive>
-            </material>
-        </xacro:macbox>
-      </link>
-      <!-- =========== WHEELS ============= -->
-        <link name="left_wheel">
-            <origin />
-            <xacro:inertialEye ma="${SIDEWHEELMASS}" mo="${SIDEWHEELMASS*.04*.04}" />
-            <xacro:maccyl radius="${WHEELRADIUS}" length="${WHEELLENGTH}" name="left_wheel">
-                <origin />
-                  <material name="rubber">
-                    <ambient>0 0 0 1</ambient>
-                  </material>
-                <surface>
-                    <friction>
-                        <ode>
-                            <mu>${WHEELSURFACEFRICTION}</mu>
-                            <mu2>${WHEELSURFACEFRICTION}</mu2>
-                            <slip1>${WHEELSURFACESLIP}</slip1>
-                            <slip2>${WHEELSURFACESLIP}</slip2>
-                        </ode>
-                    </friction>
-                </surface>
-            </xacro:maccyl>
-        </link>
-        <link name="right_wheel">
-            <origin />
-            <xacro:inertialEye ma="${SIDEWHEELMASS}" mo="${SIDEWHEELMASS*.04*.04}" />
-            <xacro:maccyl radius="${WHEELRADIUS}" length="${WHEELLENGTH}" name="right_wheel">
-                <origin />
-                  <material name="rubber">
-                    <ambient>0 0 0 1</ambient>
-                  </material>
-                <surface>
-                    <friction>
-                        <ode>
-                            <mu>${WHEELSURFACEFRICTION}</mu>
-                            <mu2>${WHEELSURFACEFRICTION}</mu2>
-                            <slip1>${WHEELSURFACESLIP}</slip1>
-                            <slip2>${WHEELSURFACESLIP}</slip2>
-                        </ode>
-                    </friction>
-                </surface>
-            </xacro:maccyl>
-        </link>
-        <link name="caster_wheel">
-            <origin />
-            <xacro:inertialEye ma="${CASTERMASS}" mo="${.695*.04*.04}" />
-            <xacro:maccyl radius="${WHEELRADIUS}" length="${WHEELLENGTH}" name="caster_wheel">
-                <origin />
-                  <material name="rubber">
-                    <ambient>0 0 0 1</ambient>
-                  </material>
-                <surface>
-                    <friction>
-                        <ode>
-                            <mu>${WHEELSURFACEFRICTION}</mu>
-                            <mu2>${WHEELSURFACEFRICTION}</mu2>
-                            <slip1>${WHEELSURFACESLIP}</slip1>
-                            <slip2>${WHEELSURFACESLIP}</slip2>
-                        </ode>
-                    </friction>
-                </surface>
-            </xacro:maccyl>
-        </link>
-        <link name="lidar_disk">
-            <origin />
-            <xacro:inertialEye ma="${LIDARMASS}" mo="${LIDARMASS*.04*.04}" />
-            <xacro:maccyl radius=".04" length=".025" name="lidar_disk">
-                <origin />
-                  <material name="rubber">
-                    <ambient>0 0 0 1</ambient>
-                  </material>
-                <surface>
-                    <friction>
-                        <ode>
-                            <mu>.9</mu>
-                            <mu2>.9</mu2>
-                            <slip1>.1</slip1>
-                            <slip2>.1</slip2>
-                        </ode>
-                    </friction>
-                </surface>
-            </xacro:maccyl>
-        </link>
-        <!-- ============= JOINTS ============== -->
-        <xacro:macro name="continuousJoint" params="name posexyz poserpy parent child xyz friction damping">
-            <joint type="continuous" name="${name}_continuous_joint">
-                <origin xyz="${posexyz}" rpy="${poserpy}"/>
-                <parent link="${parent}" />
-                <child link="${child}" />
-                <axis xyz="${xyz}" />
-                <joint_properties damping="${damping}" friction="${friction}"/>
-            </joint>
-        </xacro:macro>
-        <xacro:macro name="revoluteJoint" params="name posexyz poserpy parent child xyz friction damping lower upper effort velocity">
-            <joint type="continuous" name="${name}_revolute_joint">
-                <origin xyz="${posexyz}" rpy="${poserpy}"/>
-                <parent link="${parent}" />
-                <child link="${child}" />
-                <limit lower="${lower}" upper="${upper}" effort="${effort}" velocity="${velocity}"/>
-                <axis xyz="${xyz}" />
-                <joint_properties damping="${damping}" friction="${friction}"/>
-            </joint>
-        </xacro:macro>
-        <xacro:continuousJoint name="left_wheel"
+                <ambient>.5 .5 .5 1</ambient>
+                <diffuse>0 0 0 1</diffuse>
+                <specular>0.1 0.1 0.1 1</specular>
+                <emissive>0 0 0 0</emissive>
+            </material>
+        </xacro:macbox>
+    </link>
+    <!-- ============== WHEELS ============== -->
+    <link name="left_wheel">
+        <origin />
+        <xacro:inertialEye ma="${SIDEWHEELMASS}" mo="${SIDEWHEELMASS*.04*.04}" />
+        <xacro:maccyl radius="${WHEELRADIUS}" length="${WHEELLENGTH}" name="left_wheel">
+            <origin />
+            <material name="rubber">
+                <ambient>0 0 0 1</ambient>
+            </material>
+            <surface>
+                <friction>
+                    <ode>
+                        <mu>${WHEELSURFACEFRICTION}</mu>
+                        <mu2>${WHEELSURFACEFRICTION}</mu2>
+                        <slip1>${WHEELSURFACESLIP}</slip1>
+                        <slip2>${WHEELSURFACESLIP}</slip2>
+                    </ode>
+                </friction>
+            </surface>
+        </xacro:maccyl>
+    </link>
+    <link name="right_wheel">
+        <origin />
+        <xacro:inertialEye ma="${SIDEWHEELMASS}" mo="${SIDEWHEELMASS*.04*.04}" />
+        <xacro:maccyl radius="${WHEELRADIUS}" length="${WHEELLENGTH}" name="right_wheel">
+            <origin />
+            <material name="rubber">
+                <ambient>0 0 0 1</ambient>
+            </material>
+            <surface>
+                <friction>
+                    <ode>
+                        <mu>${WHEELSURFACEFRICTION}</mu>
+                        <mu2>${WHEELSURFACEFRICTION}</mu2>
+                        <slip1>${WHEELSURFACESLIP}</slip1>
+                        <slip2>${WHEELSURFACESLIP}</slip2>
+                    </ode>
+                </friction>
+            </surface>
+        </xacro:maccyl>
+    </link>
+    <link name="caster_wheel">
+        <origin />
+        <xacro:inertialEye ma="${CASTERMASS}" mo="${.695*.04*.04}" />
+        <xacro:maccyl radius="${WHEELRADIUS}" length="${WHEELLENGTH}" name="caster_wheel">
+            <origin />
+            <material name="rubber">
+                <ambient>0 0 0 1</ambient>
+            </material>
+            <surface>
+                <friction>
+                    <ode>
+                        <mu>${WHEELSURFACEFRICTION}</mu>
+                        <mu2>${WHEELSURFACEFRICTION}</mu2>
+                        <slip1>${WHEELSURFACESLIP}</slip1>
+                        <slip2>${WHEELSURFACESLIP}</slip2>
+                    </ode>
+                </friction>
+            </surface>
+        </xacro:maccyl>
+    </link>
+    <link name="lidar_disk">
+        <origin />
+        <xacro:inertialEye ma="${LIDARMASS}" mo="${LIDARMASS*.04*.04}" />
+        <xacro:maccyl radius=".04" length=".025" name="lidar_disk">
+            <origin />
+            <material name="rubber">
+                <ambient>0 0 0 1</ambient>
+            </material>
+            <surface>
+                <friction>
+                    <ode>
+                        <mu>.9</mu>
+                        <mu2>.9</mu2>
+                        <slip1>.1</slip1>
+                        <slip2>.1</slip2>
+                    </ode>
+                </friction>
+            </surface>
+        </xacro:maccyl>
+    </link>
+    <!-- ============== JOINTS ============== -->
+    <xacro:macro name="continuousJoint" params="name posexyz poserpy parent child xyz friction damping">
+        <joint type="continuous" name="${name}_continuous_joint">
+            <origin xyz="${posexyz}" rpy="${poserpy}"/>
+            <parent link="${parent}" />
+            <child link="${child}" />
+            <axis xyz="${xyz}" />
+            <joint_properties damping="${damping}" friction="${friction}"/>
+        </joint>
+    </xacro:macro>
+    <xacro:macro name="revoluteJoint" params="name posexyz poserpy parent child xyz friction damping lower upper effort velocity">
+        <joint type="continuous" name="${name}_revolute_joint">
+            <origin xyz="${posexyz}" rpy="${poserpy}"/>
+            <parent link="${parent}" />
+            <child link="${child}" />
+            <limit lower="${lower}" upper="${upper}" effort="${effort}" velocity="${velocity}"/>
+            <axis xyz="${xyz}" />
+            <joint_properties damping="${damping}" friction="${friction}"/>
+        </joint>
+    </xacro:macro>
+    <xacro:continuousJoint name="left_wheel"
             posexyz="0 -.12 -.11" poserpy="-${M_PI / 2} 0 0"
             parent="chassis" child="left_wheel" xyz="0 0 1"
             friction="${WHEELJOINTFRICTION}" damping="${WHEELJOINTDAMPING}" />
-        <xacro:continuousJoint name="right_wheel"
+    <xacro:continuousJoint name="right_wheel"
             posexyz="0 .12 -.11" poserpy="-${M_PI / 2} 0 0"
             parent="chassis" child="right_wheel" xyz="0 0 1"
             friction="${WHEELJOINTFRICTION}" damping="${WHEELJOINTDAMPING}" />
-        <xacro:continuousJoint name="caster_wheel"
+    <xacro:continuousJoint name="caster_wheel"
             posexyz="-.04 0 -.085" poserpy="${M_PI / 2} 0 0"
             parent="caster_arm" child="caster_wheel" xyz="0 0 1"
             friction="${WHEELJOINTFRICTION}" damping="${WHEELJOINTDAMPING}" />
-        <xacro:continuousJoint name="lidar_disk"
+    <xacro:continuousJoint name="lidar_disk"
             posexyz="0 0 .12" poserpy="0 0 0"
             parent="chassis" child="lidar_disk" xyz="0 0 1"
             friction=".001" damping=".001" />
-        <xacro:revoluteJoint name="caster_yaw"
+    <xacro:revoluteJoint name="caster_yaw"
             posexyz="-.23947 0 ${CASTERBRACKETHEIGHT}"  poserpy="0 0 0"
             parent="chassis" child="caster_arm" xyz="0 0 1"
@@ -235,15 +236,15 @@
             lower="-${M_PI}" upper="${M_PI}"
             effort="1000" velocity="1000" />
-    <!-- =================== PLUGINS ================= -->
+    <!-- ============== PLUGINS ============== -->
     <gazebo>
         <plugin name="p3d" filename="libgazebo_ros_p3d.so">
-          <alwaysOn>true</alwaysOn>
-          <bodyName>chassis</bodyName>
-          <topicName>ground_truth_p3d</topicName>
-          <serviceName>p3d_service</serviceName>
-          <gaussianNoise>0.0</gaussianNoise>
-          <updateRate>20.0</updateRate>
+            <alwaysOn>true</alwaysOn>
+            <bodyName>chassis</bodyName>
+            <topicName>ground_truth_p3d</topicName>
+            <serviceName>p3d_service</serviceName>
+            <gaussianNoise>0.0</gaussianNoise>
+            <updateRate>20.0</updateRate>
         </plugin>
-          <plugin name="differential_drive_controller" filename="libgazebo_ros_diff_drive.so">
+        <plugin name="differential_drive_controller" filename="libgazebo_ros_diff_drive.so">
             <alwaysOn>true</alwaysOn>
             <updateRate>20</updateRate>
@@ -256,6 +257,4 @@
             <leftJoint>left_wheel_continuous_joint</leftJoint>
             <rightJoint>right_wheel_continuous_joint</rightJoint>
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
Commit message: Use <gazebo> tag for surface friction.

File: description/gunnar.urdf.xacro (robot description, xacro)
@@ -24,5 +24,5 @@
         </visual>
     </xacro:macro>
-    <xacro:macro name="maccyl" params="radius length name *origin *material *surface">
+    <xacro:macro name="maccyl" params="radius length name *origin *material">
         <collision name="${name}_collision">
             <xacro:insert_block name="origin" />
@@ -30,5 +30,4 @@
                 <cylinder radius="${radius}" length="${length}" />
             </geometry>
-            <xacro:insert_block name="surface"/>
         </collision>
         <visual name="${name}_visual">
@@ -89,5 +88,4 @@
             <origin xyz="0 0 0" />
             <material  name="steel"/>
-            <surface />
         </xacro:maccyl>
         <xacro:property name="CASTERARMX" value="-.04053" />
@@ -122,16 +120,10 @@
                 <ambient>0 0 0 1</ambient>
             </material>
-            <surface>
-                <friction>
-                    <ode>
-                        <mu>${WHEELSURFACEFRICTION}</mu>
-                        <mu2>${WHEELSURFACEFRICTION}</mu2>
-                        <slip1>${WHEELSURFACESLIP}</slip1>
-                        <slip2>${WHEELSURFACESLIP}</slip2>
-                    </ode>
-                </friction>
-            </surface>
-        </xacro:maccyl>
-    </link>
+        </xacro:maccyl>
+    </link>
+    <gazebo reference="left_wheel">
+        <mu1>${WHEELSURFACEFRICTION}</mu1>
+        <mu2>${WHEELSURFACEFRICTION}</mu2>
+    </gazebo>
     <link name="right_wheel">
         <origin />
@@ -142,16 +134,10 @@
                 <ambient>0 0 0 1</ambient>
             </material>
-            <surface>
-                <friction>
-                    <ode>
-                        <mu>${WHEELSURFACEFRICTION}</mu>
-                        <mu2>${WHEELSURFACEFRICTION}</mu2>
-                        <slip1>${WHEELSURFACESLIP}</slip1>
-                        <slip2>${WHEELSURFACESLIP}</slip2>
-                    </ode>
-                </friction>
-            </surface>
-        </xacro:maccyl>
-    </link>
+        </xacro:maccyl>
+    </link>
+     <gazebo reference="right_wheel">
+        <mu1>${WHEELSURFACEFRICTION}</mu1>
+        <mu2>${WHEELSURFACEFRICTION}</mu2>
+    </gazebo>
     <link name="caster_wheel">
         <origin />
@@ -162,16 +148,10 @@
                 <ambient>0 0 0 1</ambient>
             </material>
-            <surface>
-                <friction>
-                    <ode>
-                        <mu>${WHEELSURFACEFRICTION}</mu>
-                        <mu2>${WHEELSURFACEFRICTION}</mu2>
-                        <slip1>${WHEELSURFACESLIP}</slip1>
-                        <slip2>${WHEELSURFACESLIP}</slip2>
-                    </ode>
-                </friction>
-            </surface>
-        </xacro:maccyl>
-    </link>
+        </xacro:maccyl>
+    </link>
+    <gazebo reference="caster_wheel">
+        <mu1>${WHEELSURFACEFRICTION}</mu1>
+        <mu2>${WHEELSURFACEFRICTION}</mu2>
+    </gazebo>
     <link name="lidar_disk">
         <origin />
@@ -182,14 +162,4 @@
                 <ambient>0 0 0 1</ambient>
             </material>
-            <surface>
-                <friction>
-                    <ode>
-                        <mu>.9</mu>
-                        <mu2>.9</mu2>
-                        <slip1>.1</slip1>
-                        <slip2>.1</slip2>
-                    </ode>
-                </friction>
-            </surface>
         </xacro:maccyl>
     </link>

Commit message: Correctly apply joint friction.

File: description/gunnar.urdf.xacro (robot description, xacro)
@@ -171,5 +171,5 @@
             <child link="${child}" />
             <axis xyz="${xyz}" />
-            <joint_properties damping="${damping}" friction="${friction}"/>
+            <dynamics damping="${damping}" friction="${friction}"/>
         </joint>
     </xacro:macro>
@@ -181,5 +181,5 @@
             <limit lower="${lower}" upper="${upper}" effort="${effort}" velocity="${velocity}"/>
             <axis xyz="${xyz}" />
-            <joint_properties damping="${damping}" friction="${friction}"/>
+            <dynamics damping="${damping}" friction="${friction}"/>
         </joint>
     </xacro:macro>
